Commit message: PointCloud Changes

File: Assets/URDF/niryo_one/niryo_one.urdf (robot description, URDF)
Before this commit: robot niryo_one, 15 links, 13 joints
Links:
- added link left_camera, mass 1e-5; collision box size=0.02 0.02 0.02; visual box size=0.02 0.02 0.02
- added link right_camera, mass 1e-5; collision box size=0.02 0.02 0.02; visual box size=0.02 0.02 0.02
Joints:
- added joint left_camera_joint: type fixed, parent hand_link, child left_camera, origin xyz=0.02 0.02 0.055 rpy=0 0 0, axis 0 1 0
- added joint right_camera_joint: type fixed, parent hand_link, child right_camera, origin xyz=-0.02 0.02 0.055 rpy=0 0 0, axis 0 1 0
