Commit message: Removed devel and logs. Added jointstate pub. Added funcionality to move robot. Corrected transforms

File: workspace/src/niryo_one_ros/niryo_one_description/urdf/v1/niryo_one.urdf.xacro (robot description, xacro)
@@ -217,6 +217,6 @@
     </joint>
     <joint name="left_camera_joint" type="fixed">
-        <axis xyz="0 1 0" />
-        <origin rpy="0 1.57 0" xyz="0.02 0.02 0.055" />
+        <axis xyz="1 0 0" />
+        <origin rpy="0 3.14 0" xyz="0.02 0.02 0.055" />
         <parent link="hand_link" />
         <child link="left_camera" />
@@ -243,6 +243,6 @@
     </link>
     <joint name="right_camera_joint" type="fixed">
-        <axis xyz="0 1 0" />
-        <origin rpy="0 1.57 0" xyz="-0.02 0.02 0.055" />
+        <axis xyz="1 0 0" />
+        <origin rpy="0 3.14 0" xyz="-0.02 0.02 0.055" />
         <parent link="hand_link" />
         <child link="right_camera" />

Commit message: more fixes to republisher filtering out surroundings that shouldn't be included.

File: workspace/src/niryo_one_ros/niryo_one_description/urdf/v1/niryo_one.urdf.xacro (robot description, xacro)
@@ -218,5 +218,5 @@
     <joint name="left_camera_joint" type="fixed">
         <axis xyz="1 0 0" />
-        <origin rpy="0 3.14 0" xyz="0.02 0.02 0.055" />
+        <origin rpy="3.14 3.14 0" xyz="0.02 0.02 0.055" />
         <parent link="hand_link" />
         <child link="left_camera" />
@@ -244,5 +244,5 @@
     <joint name="right_camera_joint" type="fixed">
         <axis xyz="1 0 0" />
-        <origin rpy="0 3.14 0" xyz="-0.02 0.02 0.055" />
+        <origin rpy="3.14 3.14 0" xyz="-0.02 0.02 0.055" />
         <parent link="hand_link" />
         <child link="right_camera" />
